File: schematics.and.layout/main-board.sch (EAGLE design)
At the start: 26 parts, among them U2 TPS65131

Commit message: Updated texas-instruments.lbr with LM137000. Added keyboard oscillator to schematic.
Parts:
- added C11, C12: 0.01u, rcl:C-USC0805
- added C13, C14: 1n, rcl:C-USC0805
- added R5: 1.3M, rcl:R-US_R0805
- added R7, R9: 100k, rcl:R-US_R0805
- added R8: 10k, rcl:R-US_R0805
- added U3: LM13700, texas-instruments:LM13700
- R6: value 1.3M -> 30k
Connections:
- new net KEY_OSC: C14.2
- new net N$12: R6.2, U3.INPUT_BIAS1
- new net N$13: C13.1, R9.1, U3.INPUT1-
- new net N$15: R7.2, R8.2, U3.INPUT1+
- new net N$16: C14.1, R7.1, R9.2, U3.OUTPUT1
- net +15V: now also C12.1, U3.V+
- net -15V: now also C11.2, R5.2, U3.V-; no longer R6.2
- net GND: now also C11.1, C12.2, C13.2, R6.1, R8.1
- net N$8: now also R5.1; no longer R6.1
Changed lines of the file:
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@@
 <part name="SUPPLY2" library="supply2" deviceset="GND" device=""/>
 <part name="R4" library="rcl" deviceset="R-US_" device="R0805" value="100k"/>
-<part name="R6" library="rcl" deviceset="R-US_" device="R0805" value="1.3M"/>
+<part name="R5" library="rcl" deviceset="R-US_" device="R0805" value="1.3M"/>
 <part name="C2" library="rcl" deviceset="C-US" device="C0805" value="5.7p / 25V"/>
 <part name="C3" library="rcl" deviceset="C-US" device="C0805" value="100u / 35V"/>
@@
 <part name="SUPPLY9" library="supply2" deviceset="GND" device=""/>
 <part name="C10" library="rcl" deviceset="C-US" device="C0805" value="6.8p / 25V"/>
+<part name="U3" library="texas-instruments" deviceset="LM13700" device=""/>
+<part name="R6" library="rcl" deviceset="R-US_" device="R0805" value="30k"/>
+<part name="SUPPLY10" library="supply2" deviceset="GND" device=""/>
+<part name="SUPPLY11" library="supply2" deviceset="-15V" device=""/>
+<part name="SUPPLY12" library="supply2" deviceset="+15V" device=""/>
+<part name="R7" library="rcl" deviceset="R-US_" device="R0805" value="100k"/>
+<part name="R8" library="rcl" deviceset="R-US_" device="R0805" value="10k"/>
+<part name="C11" library="rcl" deviceset="C-US" device="C0805" value="0.01u"/>
+<part name="C12" library="rcl" deviceset="C-US" device="C0805" value="0.01u"/>
+<part name="SUPPLY13" library="supply2" deviceset="GND" device=""/>
+<part name="R9" library="rcl" deviceset="R-US_" device="R0805" value="100k"/>
+<part name="C13" library="rcl" deviceset="C-US" device="C0805" value="1n"/>
+<part name="C14" library="rcl" deviceset="C-US" device="C0805" value="1n"/>
 </parts>
 <sheets>
@@
 <instance part="SUPPLY2" gate="GND" x="111.76" y="45.72"/>
 <instance part="R4" gate="G$1" x="208.28" y="68.58"/>
-<instance part="R6" gate="G$1" x="223.52" y="68.58"/>
+<instance part="R5" gate="G$1" x="223.52" y="68.58"/>
 <instance part="C2" gate="G$1" x="238.76" y="66.04"/>
 <instance part="C3" gate="G$1" x="254" y="66.04"/>
@@
 <pinref part="R4" gate="G$1" pin="2"/>
 <wire x1="213.36" y1="68.58" x2="215.9" y2="68.58" width="0.1524" layer="91"/>
-<pinref part="R6" gate="G$1" pin="1"/>
+<pinref part="R5" gate="G$1" pin="1"/>
 <pinref part="U2" gate="A" pin="FBN"/>
 <wire x1="215.9" y1="68.58" x2="218.44" y2="68.58" width="0.1524" layer="91"/>
@@
 <wire x1="215.9" y1="58.42" x2="231.14" y2="58.42" width="0.1524" layer="91"/>
 <wire x1="231.14" y1="58.42" x2="231.14" y2="68.58" width="0.1524" layer="91"/>
-<pinref part="R6" gate="G$1" pin="2"/>
+<pinref part="R5" gate="G$1" pin="2"/>
 <wire x1="231.14" y1="68.58" x2="228.6" y2="68.58" width="0.1524" layer="91"/>
 <wire x1="231.14" y1="58.42" x2="238.76" y2="58.42" width="0.1524" layer="91"/>
@@
 </segment>
 </net>
+</nets>
+</sheet>
+<sheet>
+<plain>
+</plain>
+<instances>
+<instance part="U3" gate="G$1" x="68.58" y="48.26"/>
+<instance part="R6" gate="G$1" x="2.54" y="60.96" rot="R90"/>
+<instance part="SUPPLY10" gate="GND" x="2.54" y="27.94"/>
+<instance part="SUPPLY11" gate="G$1" x="25.4" y="27.94"/>
+<instance part="SUPPLY12" gate="+15V" x="104.14" y="45.72"/>
+<instance part="R7" gate="G$1" x="33.02" y="55.88"/>
+<instance part="R8" gate="G$1" x="22.86" y="60.96"/>
+<instance part="C11" gate="G$1" x="17.78" y="33.02" rot="R90"/>
+<instance part="C12" gate="G$1" x="104.14" y="35.56"/>
+<instance part="SUPPLY13" gate="GND" x="104.14" y="25.4"/>
+<instance part="R9" gate="G$1" x="22.86" y="45.72"/>
+<instance part="C13" gate="G$1" x="10.16" y="43.18"/>
+<instance part="C14" gate="G$1" x="33.02" y="35.56"/>
+</instances>
+<busses>
+</busses>
+<nets>
+<net name="N$12" class="0">
+<segment>
+<pinref part="R6" gate="G$1" pin="2"/>
+<pinref part="U3" gate="G$1" pin="INPUT_BIAS1"/>
+<wire x1="2.54" y1="66.04" x2="43.18" y2="66.04" width="0.1524" layer="91"/>
+</segment>
+</net>
+<net name="GND" class="0">
+<segment>
+<pinref part="SUPPLY10" gate="GND" pin="GND"/>
+<pinref part="R6" gate="G$1" pin="1"/>
+<wire x1="2.54" y1="30.48" x2="2.54" y2="33.02" width="0.1524" layer="91"/>
+<wire x1="2.54" y1="33.02" x2="2.54" y2="45.72" width="0.1524" layer="91"/>
+<pinref part="C11" gate="G$1" pin="1"/>
+<wire x1="2.54" y1="45.72" x2="2.54" y2="55.88" width="0.1524" layer="91"/>
+<wire x1="15.24" y1="33.02" x2="10.16" y2="33.02" width="0.1524" layer="91"/>
+<junction x="2.54" y="33.02"/>
+<pinref part="R8" gate="G$1" pin="1"/>
+<wire x1="10.16" y1="33.02" x2="2.54" y2="33.02" width="0.1524" layer="91"/>
+<wire x1="17.78" y1="60.96" x2="7.62" y2="60.96" width="0.1524" layer="91"/>
+<wire x1="7.62" y1="60.96" x2="7.62" y2="45.72" width="0.1524" layer="91"/>
+<wire x1="7.62" y1="45.72" x2="2.54" y2="45.72" width="0.1524" layer="91"/>
+<junction x="2.54" y="45.72"/>
+<pinref part="C13" gate="G$1" pin="2"/>
+<wire x1="10.16" y1="38.1" x2="10.16" y2="33.02" width="0.1524" layer="91"/>
+<junction x="10.16" y="33.02"/>
+</segment>
+<segment>
+<pinref part="SUPPLY13" gate="GND" pin="GND"/>
+<pinref part="C12" gate="G$1" pin="2"/>
+<wire x1="104.14" y1="27.94" x2="104.14" y2="30.48" width="0.1524" layer="91"/>
+</segment>
+</net>
+<net name="+15V" class="0">
+<segment>
+<pinref part="U3" gate="G$1" pin="V+"/>
+<pinref part="SUPPLY12" gate="+15V" pin="+15V"/>
+<wire x1="93.98" y1="40.64" x2="104.14" y2="40.64" width="0.1524" layer="91"/>
+<wire x1="104.14" y1="40.64" x2="104.14" y2="43.18" width="0.1524" layer="91"/>
+<pinref part="C12" gate="G$1" pin="1"/>
+<wire x1="104.14" y1="38.1" x2="104.14" y2="40.64" width="0.1524" layer="91"/>
+<junction x="104.14" y="40.64"/>
+</segment>
+</net>
+<net name="-15V" class="0">
+<segment>
+<pinref part="U3" gate="G$1" pin="V-"/>
+<pinref part="SUPPLY11" gate="G$1" pin="-15V"/>
+<wire x1="43.18" y1="40.64" x2="25.4" y2="40.64" width="0.1524" layer="91"/>
+<wire x1="25.4" y1="40.64" x2="25.4" y2="33.02" width="0.1524" layer="91"/>
+<pinref part="C11" gate="G$1" pin="2"/>
+<wire x1="25.4" y1="33.02" x2="25.4" y2="30.48" width="0.1524" layer="91"/>
+<wire x1="22.86" y1="33.02" x2="25.4" y2="33.02" width="0.1524" layer="91"/>
+<junction x="25.4" y="33.02"/>
+</segment>
+</net>
+<net name="N$15" class="0">
+<segment>
+<pinref part="R7" gate="G$1" pin="2"/>
+<pinref part="U3" gate="G$1" pin="INPUT1+"/>
+<wire x1="38.1" y1="55.88" x2="40.64" y2="55.88" width="0.1524" layer="91"/>
+<pinref part="R8" gate="G$1" pin="2"/>
+<wire x1="40.64" y1="55.88" x2="43.18" y2="55.88" width="0.1524" layer="91"/>
+<wire x1="27.94" y1="60.96" x2="40.64" y2="60.96" width="0.1524" layer="91"/>
+<wire x1="40.64" y1="60.96" x2="40.64" y2="55.88" width="0.1524" layer="91"/>
+<junction x="40.64" y="55.88"/>
+</segment>
+</net>
+<net name="N$16" class="0">
+<segment>
+<pinref part="R7" gate="G$1" pin="1"/>
+<pinref part="U3" gate="G$1" pin="OUTPUT1"/>
+<wire x1="27.94" y1="45.72" x2="33.02" y2="45.72" width="0.1524" layer="91"/>
+<wire x1="33.02" y1="45.72" x2="43.18" y2="45.72" width="0.1524" layer="91"/>
+<wire x1="27.94" y1="55.88" x2="27.94" y2="45.72" width="0.1524" layer="91"/>
+<pinref part="R9" gate="G$1" pin="2"/>
+<junction x="27.94" y="45.72"/>
+<pinref part="C14" gate="G$1" pin="1"/>
+<wire x1="33.02" y1="38.1" x2="33.02" y2="45.72" width="0.1524" layer="91"/>
+<junction x="33.02" y="45.72"/>
+</segment>
+</net>
+<net name="N$13" class="0">
+<segment>
+<pinref part="U3" gate="G$1" pin="INPUT1-"/>
+<pinref part="R9" gate="G$1" pin="1"/>
+<wire x1="43.18" y1="50.8" x2="17.78" y2="50.8" width="0.1524" layer="91"/>
+<wire x1="17.78" y1="50.8" x2="17.78" y2="45.72" width="0.1524" layer="91"/>
+<pinref part="C13" gate="G$1" pin="1"/>
+<wire x1="10.16" y1="45.72" x2="10.16" y2="50.8" width="0.1524" layer="91"/>
+<wire x1="10.16" y1="50.8" x2="17.78" y2="50.8" width="0.1524" layer="91"/>
+<junction x="17.78" y="50.8"/>
+</segment>
+</net>
+<net name="KEY_OSC" class="0">
+<segment>
+<pinref part="C14" gate="G$1" pin="2"/>
+<wire x1="33.02" y1="30.48" x2="33.02" y2="17.78" width="0.1524" layer="91"/>
+<wire x1="33.02" y1="17.78" x2="45.72" y2="17.78" width="0.1524" layer="91"/>
+<label x="45.72" y="17.78" size="1.778" layer="95"/>
+</segment>
+</net>
